File: HDMI_DVI_DISP_7/HDMI_DVI_DISP_7.kicad_pcb (KiCad board)
At the start: 4 copper layers, 169 parts, among them J201 HDMI_A, J202 Jack-DC, J203 Conn_01x40_MountingPin, Q401 SiA453EDJ, Q402 MUN5211DW1, SW301 DM-05-V, U201 ADG633YCP, U202 24LC32, U203 LP2985-3.3, U204 TXB0102DCT, U301 TFP401A, U302 SN65LVDS93A, U401 TPS54286

Commit message: Major progress of PCB layout
Parts:
- added C317: 68n, Capacitor_SMD:C_0402_1005Metric, B.Cu at (70.7, 82.2)
- C301, C302, C303, C304, C305, C306, C307, C308: moved to B.Cu
- moved C302 174.8 mm to (55.3, 95.7), turned to 90 degrees
- moved C303 170.4 mm to (62.7, 104.1), turned to 270 degrees
- moved C304 159.6 mm to (65.0, 104.1), turned to 270 degrees
- moved C310 159.1 mm to (59.7, 92.9), turned to 270 degrees
- moved C306 158.8 mm to (70.2, 104.1), turned to 270 degrees
- moved C308 155.6 mm to (76.4, 95.8)
- moved C305 154.3 mm to (55.3, 90.7), turned to 90 degrees
- moved FB303 150.8 mm to (57.1, 102.0), turned to 90 degrees
- moved C311 148.6 mm to (55.1, 101.8), turned to 90 degrees
- moved C307 147.2 mm to (75.5, 89.7)
- moved FB302 137.6 mm to (59.7, 88.6), turned to 90 degrees
- moved C301 137.2 mm to (60.2, 82.3), turned to 90 degrees
- moved FB304 137.0 mm to (70.3, 87.5)
- moved C325 134.2 mm to (102.8, 98.1), turned to 270 degrees
- moved C324 132.8 mm to (102.8, 105.2), turned to 270 degrees
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Connections:
- net Net-(U301-Pad10) renamed /900_Video_Links/QE0
- net Net-(U301-Pad11) renamed /900_Video_Links/QE1
- net Net-(U301-Pad12) renamed /900_Video_Links/QE2
- net Net-(U301-Pad13) renamed /900_Video_Links/QE3
- net Net-(U301-Pad14) renamed /900_Video_Links/QE4
- net Net-(U301-Pad15) renamed /900_Video_Links/QE5
- net Net-(U301-Pad16) renamed /900_Video_Links/QE6
- net Net-(U301-Pad17) renamed /900_Video_Links/QE7
- net Net-(U301-Pad20) renamed /900_Video_Links/QE8
- net Net-(U301-Pad21) renamed /900_Video_Links/QE9
- net Net-(U301-Pad22) renamed /900_Video_Links/QE10
- net Net-(U301-Pad23) renamed /900_Video_Links/QE11
- net Net-(U301-Pad24) renamed /900_Video_Links/QE12
- net Net-(U301-Pad25) renamed /900_Video_Links/QE13
- net Net-(U301-Pad26) renamed /900_Video_Links/QE14
- net Net-(U301-Pad27) renamed /900_Video_Links/QE15
- net Net-(U301-Pad30) renamed /900_Video_Links/QE16
- net Net-(U301-Pad31) renamed /900_Video_Links/QE17
- net Net-(U301-Pad32) renamed /900_Video_Links/QE18
- net Net-(U301-Pad33) renamed /900_Video_Links/QE19
- net Net-(U301-Pad34) renamed /900_Video_Links/QE20
- net Net-(U301-Pad35) renamed /900_Video_Links/QE21
- net Net-(U301-Pad36) renamed /900_Video_Links/QE22
- net Net-(U301-Pad37) renamed /900_Video_Links/QE23
- net Net-(U301-Pad44) renamed /900_Video_Links/ODCK
- net Net-(U301-Pad46) renamed /900_Video_Links/DE
- net Net-(U301-Pad47) renamed /900_Video_Links/VSYNC
- net Net-(U301-Pad48) renamed /900_Video_Links/HSYNC
Routing:
- net /900_Video_Links/P_TMDS_OVDD_3V3: track 0.00 -> 76.6 mm, vias 0 -> 6
- net /900_Video_Links/QE11: track 0.00 -> 53.2 mm, vias 0 -> 2
- net /900_Video_Links/QE14: track 0.00 -> 53.2 mm
- net /900_Video_Links/QE15: track 0.00 -> 53.2 mm, vias 0 -> 2
- net /900_Video_Links/QE13: track 0.00 -> 53.2 mm
- net /900_Video_Links/DE: track 0.00 -> 53.2 mm, vias 0 -> 3
- net /900_Video_Links/QE18: track 0.00 -> 53.1 mm, vias 0 -> 3
- net /900_Video_Links/QE19: track 0.00 -> 53.1 mm, vias 0 -> 2
- net /900_Video_Links/QE2: track 0.00 -> 53.1 mm, vias 0 -> 2
- net /900_Video_Links/QE0: track 0.00 -> 53.1 mm, vias 0 -> 3
- net /900_Video_Links/QE9: track 0.00 -> 53.1 mm, vias 0 -> 2
- net /900_Video_Links/QE16: track 0.00 -> 53.1 mm, vias 0 -> 3
- net /900_Video_Links/QE3: track 0.00 -> 53.1 mm, vias 0 -> 2
- net /900_Video_Links/QE6: track 0.00 -> 53.1 mm, vias 0 -> 2
- net /900_Video_Links/QE21: track 0.00 -> 53.1 mm
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